File: ardf144.kicad_pcb (KiCad board)
At the start: 2 copper layers, 146.7 x 39.4 mm, 54 parts, among them J1 Jack-DC, Q1 2SC1906, SW1 SW_SPST, U1 NE612, U2 2SK439, U3 L7805, U4 LM386, U5 2SK439, Y1 16MHz

Commit message: second
Parts:
- added J2: Conn_01x02_Socket, Connector_PinSocket_2.54mm:PinSocket_1x02_P2.54mm_Vertical, F.Cu at (177.7, 61.3)
- added J3: Conn_01x02_Socket, Connector_PinSocket_2.54mm:PinSocket_1x02_P2.54mm_Vertical, F.Cu at (79.5, 49.5)
- C9: footprint Capacitor_THT:C_Disc_D5.0mm_W2.5mm_P2.50mm -> Capacitor_THT:CP_Radial_D6.3mm_P2.50mm
- J1: footprint Connector_BarrelJack:BarrelJack_Wuerth_694106106102_2.0x5.5mm -> Library:2.5jack
- moved J1 35.9 mm to (175.7, 39.8), turned to 0 degrees
- moved C8 20.1 mm to (86.3, 56.4)
- moved C9 18.2 mm to (91.3, 59.1)
- moved C11 17.2 mm to (153.2, 48.8), turned to -90 degrees
- moved R7 16.8 mm to (170.1, 48.1), turned to 0 degrees
- moved U3 15.4 mm to (104.6, 60.8)
- moved C14 11.4 mm to (175.2, 53.5)
- moved C16 8.50 mm to (163.8, 52.5)
- moved C2 8.21 mm to (107.0, 41.1), turned to 0 degrees
- moved RV2 6.29 mm to (126.0, 61.2)
- moved R6 6.25 mm to (154.2, 58.2)
- moved C17 5.46 mm to (169.6, 36.7), turned to -90 degrees
- moved L2 5.21 mm to (126.2, 47.5)
- moved RV1 5.11 mm to (127.5, 38.1)
- moved C6 4.72 mm to (133.1, 42.7)
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Connections:
- C1 pad 1: unconnected-(C1-Pad1) -> Net-(J3-Pin_2)
- RV1 pad 1: 9v -> GND
- RV1 pad 3: GND -> 9v
- SW1 pad 1: unconnected-(SW1-A-Pad1) -> Net-(J2-Pin_1)
Routing:
- net Net-(U4--): track 23.3 -> 52.2 mm
- net 9v: track 157.0 -> 178.7 mm
- net Net-(U1-OSC_B): track 9.06 -> 30.3 mm
- net Lo.: track 23.7 -> 5.07 mm
- net Net-(J2-Pin_1): track 0.00 -> 8.84 mm
- net Net-(J1-Pad2): track 0.00 -> 7.83 mm
- net Net-(D1-A): track 34.7 -> 42.4 mm
- net Net-(J3-Pin_2): track 0.00 -> 5.84 mm
- net Net-(U4-V+): track 18.0 -> 12.4 mm
- net Net-(C15-Pad1): track 42.8 -> 38.0 mm
- net Net-(U2-D): track 13.6 -> 18.2 mm
- net AF: track 22.3 -> 18.5 mm
- net unconnected-(SW1-A-Pad1): track 3.30 -> 0.00 mm
- net Net-(U2-S): track 14.5 -> 11.7 mm
- net 5v: track 59.7 -> 62.4 mm
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Other:
- board size 146.7 x 39.4 mm -> 150 x 30.2 mm
