File: ardf144_2.kicad_pcb (KiCad board)
At the start: 2 copper layers, 150 x 30.2 mm, 59 parts, among them J1 Jack-DC, J2 batt, J3 ant, Q1 2SC1906, SW1 SW_SPST, U1 NE612, U2 2SK439, U3 L7805, U4 LM386, U5 2SK439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

Commit message: fix 3
Parts:
- C26: footprint Capacitor_THT:C_Disc_D5.0mm_W2.5mm_P5.00mm -> Capacitor_THT:C_Disc_D5.0mm_W2.5mm_P2.50mm
- C27: moved to F.Cu
- D2: footprint Diode_THT:D_DO-41_SOD81_P2.54mm_Vertical_AnodeUp -> Diode_THT:D_DO-41_SOD81_P10.16mm_Horizontal
- J2: value batt -> Conn_01x02_Socket
- J3: value ant -> Conn_01x02_Socket
- R7: value 10 -> R
- moved C26 29.6 mm to (134.7, 67.9), turned to 0 degrees
- moved C24 9.62 mm to (69.8, 57.2), turned to -90 degrees
- moved U3 6.86 mm to (104.6, 60.8)
- moved C27 6.82 mm to (116.9, 50.2)
- moved U5 6.35 mm to (59.1, 37.5), turned to 0 degrees
- moved C9 6.26 mm to (91.3, 59.1)
- moved L5 4.53 mm to (79.1, 57.4)
- moved R4 3.22 mm to (103.5, 53.8)
- moved R3 3.17 mm to (92.7, 44.2)
- moved C8 1.89 mm to (86.3, 56.4)
- moved L2 1.59 mm to (126.2, 47.5), turned to 0 degrees
- moved L4 0.64 mm to (63.5, 50.8)
- moved L1 0.38 mm to (100.1, 42.2)
Routing:
- net Net-(C23-Pad1): track 14.2 -> 24.1 mm
- net 9v: track 185.5 -> 178.7 mm
- net Net-(U5-G): track 5.71 -> 12.5 mm
- net Net-(U1-OUT_B): track 6.50 -> 0.00 mm
- net Net-(U1-IN_B): track 24.4 -> 18.2 mm
- net Lo.: track 10.5 -> 5.07 mm
- net Net-(C4-Pad1): track 19.9 -> 15.6 mm
- net Net-(U1-IN_A): track 8.87 -> 12.1 mm
- net Net-(U2-D): track 16.4 -> 18.2 mm
- net Net-(C23-Pad2): track 11.5 -> 13.2 mm
- net Net-(L1-Pad2): track 9.52 -> 8.13 mm
- net Net-(U1-OSC_B): track 31.7 -> 30.3 mm
- net Net-(U5-D): track 5.08 -> 3.81 mm
- net Net-(Q1-C): track 28.0 -> 27.2 mm
- net Net-(D1-A): track 42.9 -> 42.4 mm
