File: ic4ardf.kicad_pcb (KiCad board)
At the start: 2 copper layers, 26 parts, among them J1 Conn_Coaxial, J2 Barrel_Jack, SW1 SW_SPDT_312, U1 tiny85, U2 Si5351, U3 SA612, U4 LM386, U5 LM78L05_TO92, U6 L78L33_TO92

Commit message: fix attiny vcc +3v3 from +5v
Parts:
- U1: value tiny85 -> ATtiny85-20P
- U2: value Si5351 -> Si5351module
Connections:
- U1 pad 8: +5V -> +3V3
Routing:
- net GND: track 141.9 -> 149.0 mm
- net +5V: track 60.2 -> 57.1 mm
- net +3V3: track 36.2 -> 33.7 mm
Changed lines of the file:
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@@
 			)
 		)
-		(property "Value" "tiny85"
+		(property "Value" "ATtiny85-20P"
 			(at 3.81 5.07 0)
 			(layer "F.Fab")
@@
 			(layers "*.Cu" "*.Mask")
 			(remove_unused_layers no)
-			(net 20 "+5V")
+			(net 25 "+3V3")
 			(pinfunction "VCC")
 			(pintype "power_in")
@@
 		(tags "Potentiometer vertical Vishay T73YP")
 		(property "Reference" "RV1"
-			(at -0.06 -7.09 270)
+			(at -0.06 -7.09 -90)
 			(layer "F.SilkS")
 			(effects
@@
 		)
 		(property "Value" "10k"
-			(at -0.06 2.01 270)
+			(at -0.06 2.01 -90)
 			(layer "F.Fab")
 			(effects
@@
 		)
 		(fp_text user "${REFERENCE}"
-			(at -2.56 -2.54 360)
+			(at -2.56 -2.54 0)
 			(layer "F.Fab")
 			(effects
@@
 			)
 		)
-		(property "Value" "Si5351"
+		(property "Value" "Si5351module"
 			(at 3.81 5.08 0)
 			(layer "F.Fab")
@@
 		(tags "C Disc series Radial pin pitch 5.00mm  diameter 4.3mm width 1.9mm Capacitor")
 		(property "Reference" "C13"
-			(at 2.5 -2.2 270)
+			(at 2.5 -2.2 -90)
 			(layer "F.SilkS")
 			(effects
@@
 		)
 		(property "Value" "C"
-			(at 2.5 2.2 270)
+			(at 2.5 2.2 -90)
 			(layer "F.Fab")
 			(effects
@@
 		)
 		(fp_text user "${REFERENCE}"
-			(at 2.5 0 270)
+			(at 2.5 0 -90)
 			(layer "F.Fab")
 			(effects
@@
 		(tags "CP Radial series Radial pin pitch 2.50mm  diameter 6.3mm Electrolytic Capacitor")
 		(property "Reference" "C10"
-			(at 1.25 -4.4 270)
+			(at 1.25 -4.4 -90)
 			(layer "F.SilkS")
 			(effects
@@
 		)
 		(property "Value" "C_Polarized"
-			(at 1.25 4.4 270)
+			(at 1.25 4.4 -90)
 			(layer "F.Fab")
 			(effects
@@
 		)
 		(fp_text user "${REFERENCE}"
-			(at 1.25 0 270)
+			(at 1.25 0 -90)
 			(layer "F.Fab")
 			(effects
@@
 		(tags "SMA")
 		(property "Reference" "J1"
-			(at -3.96 3 270)
+			(at -3.96 3 -90)
 			(layer "B.SilkS")
 			(effects
@@
 		)
 		(fp_text user "${REFERENCE}"
-			(at 4.79 0 270)
+			(at 4.79 0 -90)
 			(layer "B.Fab")
 			(effects
@@
 	)
 	(segment
-		(start 85.09 92.9475)
-		(end 85.09 80.645)
+		(start 106.72 76.24)
+		(end 106.68 76.2)
 		(width 0.2)
 		(layer "B.Cu")
@@
 	)
 	(segment
-		(start 83.82 73.66)
-		(end 86.72 73.66)
+		(start 106.72 96.52)
+		(end 106.72 76.24)
 		(width 0.2)
 		(layer "B.Cu")
@@
 	)
 	(segment
-		(start 104.18 93.98)
-		(end 103.380001 94.779999)
+		(start 83.82 73.66)
+		(end 86.72 73.66)
 		(width 0.2)
 		(layer "B.Cu")
@@
 	)
 	(segment
-		(start 93.99 76.21)
-		(end 95.09 77.31)
-		(width 0.2)
-		(layer "B.Cu")
-		(net 1)
-	)
-	(segment
-		(start 85.09 80.645)
-		(end 86.085 79.65)
-		(width 0.2)
-		(layer "B.Cu")
-		(net 1)
-	)
-	(segment
-		(start 104.14 86.36)
-		(end 106.72 88.94)
-		(width 0.2)
-		(layer "B.Cu")
-		(net 1)
-	)
-	(segment
 		(start 116.84 95.25)
 		(end 115.57 96.52)
@@
 	)
 	(segment
-		(start 93.99 76.21)
-		(end 91.45 76.21)
+		(start 104.18 96.52)
+		(end 85.09 96.52)
 		(width 0.2)
 		(layer "B.Cu")
@@
 	)
 	(segment
-		(start 106.72 96.52)
-		(end 104.18 93.98)
+		(start 93.99 76.21)
+		(end 91.45 76.21)
 		(width 0.2)
 		(layer "B.Cu")
@@
 	)
 	(segment
-		(start 95.09 77.31)
-		(end 103.03 77.31)
+		(start 85.09 96.52)
+		(end 85.09 80.645)
 		(width 0.2)
 		(layer "B.Cu")
@@
 	)
 	(segment
+		(start 104.14 86.36)
+		(end 106.68 86.36)
+		(width 0.2)
+		(layer "B.Cu")
+		(net 1)
+	)
+	(segment
 		(start 87.99 76.12)
 		(end 91.36 76.12)
@@
 	)
 	(segment
+		(start 104.18 96.52)
+		(end 106.72 96.52)
+		(width 0.2)
+		(layer "B.Cu")
+		(net 1)
+	)
+	(segment
 		(start 76.56 73.66)
 		(end 76.56 76.2)
@@
 	)
 	(segment
-		(start 87.99 74.97)
-		(end 88.01 74.95)
+		(start 85.09 80.645)
+		(end 86.085 79.65)
 		(width 0.2)
 		(layer "B.Cu")
@@
 	)
 	(segment
-		(start 115.57 96.52)
-		(end 106.72 96.52)
+		(start 87.99 74.97)
+		(end 88.01 74.95)
 		(width 0.2)
 		(layer "B.Cu")
@@
 	)
 	(segment
-		(start 106.72 88.94)
-		(end 106.72 96.52)
+		(start 104.14 76.2)
+		(end 106.68 76.2)
 		(width 0.2)
 		(layer "B.Cu")
@@
 	)
 	(segment
-		(start 103.380001 94.779999)
-		(end 86.922499 94.779999)
+		(start 115.57 96.52)
+		(end 106.72 96.52)
 		(width 0.2)
 		(layer "B.Cu")
@@
 	)
 	(segment
-		(start 86.922499 94.779999)
-		(end 85.09 92.9475)
+		(start 104.18 93.98)
+		(end 104.18 96.52)
 		(width 0.2)
 		(layer "B.Cu")
@@
 	)
 	(segment
-		(start 103.03 77.31)
-		(end 104.14 76.2)
-		(width 0.2)
-		(layer "B.Cu")
-		(net 1)
-	)
-	(segment
 		(start 86.085 78.025)
 		(end 87.99 76.12)
@@
 	)
 	(segment
-		(start 100.33 66.04)
-		(end 101.61 67.32)
-		(width 0.2)
-		(layer "B.Cu")
-		(net 20)
-	)
-	(segment
 		(start 111.76 81.28)
 		(end 111.76 78.74)
@@
 	)
 	(segment
-		(start 101.61 67.32)
-		(end 101.61 68.59)
-		(width 0.2)
-		(layer "B.Cu")
-		(net 20)
-	)
-	(segment
 		(start 87.99 71.12)
 		(end 87.99 66.95)
@@
 	)
 	(segment
+		(start 99.06 78.74)
+		(end 99.06 68.58)
+		(width 0.2)
+		(layer "B.Cu")
+		(net 25)
+	)
+	(segment
+		(start 99.06 68.58)
+		(end 99.07 68.59)
+		(width 0.2)
+		(layer "B.Cu")
+		(net 25)
+	)
+	(segment
+		(start 104.14 68.58)
+		(end 103.58 68.58)
+		(width 0.2)
+		(layer "B.Cu")
+		(net 25)
+	)
+	(segment
 		(start 91.44 78.74)
-		(end 106.68 78.74)
+		(end 99.06 78.74)
 		(width 0.2)
 		(layer "B.Cu")
@@
 	)
 	(segment
-		(start 106.68 78.74)
+		(start 104.14 68.58)
 		(end 106.68 68.58)
 		(width 0.2)
@@
 	)
 	(segment
-		(start 104.14 68.58)
-		(end 106.68 68.58)
+		(start 99.07 68.59)
+		(end 101.61 68.59)
+		(width 0.2)
+		(layer "B.Cu")
+		(net 25)
+	)
+	(segment
+		(start 103.58 68.58)
+		(end 103.57 68.59)
+		(width 0.2)
+		(layer "B.Cu")
+		(net 25)
+	)
+	(segment
+		(start 103.57 68.59)
+		(end 101.61 68.59)
 		(width 0.2)
 		(layer "B.Cu")
